File: eps/hardware/eps.kicad_sch (KiCad schematic)
At the start: 0 parts

Commit message: begin implementing battery charger
Changed lines of the file:
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@@
 			)
 		)
-		(property "Value" "V+"
-			(at 52.07 17.78 0)
+		(property "Value" "VIN"
+			(at 54.61 21.5899 0)
 			(effects
 				(font
 					(size 1.27 1.27)
 				)
+				(justify left)
 			)
 		)
